Commit message: Model fix + full PID tuning system

File: models/robot/rescue-float-robot/robot.urdf (robot description, URDF)
Before this commit: robot C:\Users\Admin\rescue-float-robot, 3 links, 2 joints
Joints:
- joint leftmotor: limit lower=-3.141592653589793 upper=3.141592653589793 effort=10 velocity=10 -> effort=10 velocity=10; type revolute -> continuous
- joint rightmotor: limit lower=-3.141592653589793 upper=3.141592653589793 effort=10 velocity=10 -> effort=10 velocity=10; type revolute -> continuous
